File: pcb/hub.kicad_sch (KiCad schematic)
At the start: 21 parts, among them U3 USB2514B, Y2 24MHz

Commit message: derive the hub's crystal load properly, and correct what I said about it
The hub's loading capacitors imply a 10 pF crystal, not the 12 pF recorded yesterday. The error was
in the arithmetic, and it is worth writing down because the obvious way to do it is wrong: stray
capacitance sits in parallel with each loading capacitor, not with the two of them in series, so
the load is not half the pair plus the stray but half of the pair-plus-the-stray. With the 18 pF
the hub's own documents call typical and a few picofarads of board stray that is about 10.5 pF.
The naive route gives 12 pF, which is a different part to buy. Both of the vendor's formulations,
the older datasheet's and the newer checklist's, agree once read carefully.

The frequency allowance is a trap in the other direction. The +/-350 ppm quoted is the total the
hub tolerates, so a part sold as +/-350 ppm spends the whole budget before temperature and ageing;
the field now asks for a commodity +/-50 ppm, which meets it several times over.

The 1 Mohm the datasheet figure draws across the crystal is not ours to fit. The design checklist
exists to list what the board must provide and asks only for the two loading capacitors. It also
confirms two things already drawn: the 12.0k 1% reference to ground, and that the hub's reset may
be held by the processor rather than pulled up, which is what the pull-down and the GPIO on it
amount to.

I also said those two documents were scanned images that nothing could be read out of. They are
not; my own reader fails on them where the renderer's text extraction does not, which is a fact
about the reader rather than the files.

Co-Authored-By: Claude Opus 5 (1M context) <noreply@anthropic.com>
Parts:
- Y2: Load 12pF -> 10pF; Tolerance 30ppm -> 50ppm
Changed lines of the file:
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@@
 			)
 		)
-		(property "Tolerance" "30ppm"
+		(property "Tolerance" "50ppm"
 			(at 137.16 144.78 0)
 			(show_name no)
@@
 			)
 		)
-		(property "Load" "12pF"
+		(property "Load" "10pF"
 			(at 137.16 144.78 0)
 			(show_name no)
