File: pcb/hub.kicad_sch (KiCad schematic)
At the start: 21 parts, among them U3 USB2514B, Y2 24MHz

Commit message: manual pcb finishing work
Parts:
- renumbered C34 to C29, C35 to C30, C36 to C31, C37 to C33, C38 to C34, C33 to C35, C39 to C36, C30 to C37, C31 to C38, R26 to R12, R27 to R13, R28 to R14, R24 to R15, R25 to R16, R23 to R17, R20 to R18, R21 to R19, R22 to R20, U3 to U5
