File: pcb/hub.kicad_sch (KiCad schematic)
At the start: 24 parts, among them U5 USB2514B, Y2 24MHz

Commit message: settle the open items by reading, pick the fabricator, and script the export
The flash is rated 133 MHz for everything but the plain read, so the QSPI divider's 120 MHz
stands. The buck's values are checked against its datasheet's table and text: the 4.7 uH stays
inside the recommended band with 0.22 A of ripple; the input capacitor becomes the same 10 uF 0805
16 V X7R part as the hub's bulk capacitor, so it still reads 10 uF with 5 V across it; the inductor
is named, a Coilcraft XEL4030-472MEC on the land already placed, chosen over the XFL part in the
same size because that one saturates below the buck's current limit. VBUS carries 10.6 uF nominal
and about 8 uF real at attach, under the 10 uF allowed. The three items that only a prototype can
answer move to their own list, with the crystals' drive level added to it.

The board goes to JLCPCB assembled: four layers with 0.2 mm vias is its standard process, it fills
and caps vias in pads, it assembles both faces and through-hole, and the four chips that matter
are in its catalogue -- their numbers are now LCSC fields on the symbols and a column in the bill
of materials. The two connectors are not, and go in as sourced or consigned parts.

scripts/export-fab.ps1 writes the Gerber and drill zip, the bill of materials and the placement
file to pcb/fab/ (untracked), after a rules check with schematic parity that refills the pours and
saves the board first, since the Gerbers are plotted from the stored fill. The first run found the
fill a step behind the last edit, which the saved board now carries.

The board still has the old C20 footprint and lacks the new fields until the schematic is pushed
to it, which is the next step before the export passes.

Co-Authored-By: Claude Fable 5.1 <noreply@anthropic.com>
Parts:
- U5: LCSC (none) -> C16251; MPN (none) -> USB2514B-AEZC-TR
Changed lines of the file:
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@@
+			)
+		)
+		(property "MPN" "USB2514B-AEZC-TR"
+			(at 205.3433 167.64 0)
+			(show_name no)
+			(do_not_autoplace no)
+			(hide yes)
+			(effects
+				(font
+					(size 1.27 1.27)
+				)
+				(justify left)
+			)
+		)
+		(property "LCSC" "C16251"
+			(at 205.3433 167.64 0)
+			(show_name no)
+			(do_not_autoplace no)
+			(hide yes)
+			(effects
+				(font
+					(size 1.27 1.27)
+				)
+				(justify left)
 			)
 		)

Commit message: every bill-of-materials line answers the assembler
The first upload to the fabricator matched the passives by value and package and failed nine
lines. Each line now carries a definite answer in the schematic, written out as columns: a
catalogue number where the part is in the catalogue -- the flash, the protection arrays, the
indicators, the ferrite, and both crystals as 10 pF parts, since the catalogue's basic crystals
are 20 pF and the processor vendor's circuit was copied with its 15 pF capacitors; a named part
and a global-sourcing note where it is not -- the buck inductor, the buttons, the USB-C receptacle
and the USB-A sockets. The debug header is marked not fitted, and the mounting holes leave the
bill and the placement file, since neither is a part.

The same fields are on the board's footprints, as an update from the schematic would put them, so
parity holds; the export writes the sourcing column; the design document carries the table.

Co-Authored-By: Claude Fable 5.1 <noreply@anthropic.com>
Parts:
- Y2: LCSC (none) -> C70583; MPN (none) -> YXC X322524MMB4SI
Changed lines of the file:
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@@
+			)
+		)
+		(property "LCSC" "C70583"
+			(at 137.16 137.16 0)
+			(show_name no)
+			(do_not_autoplace no)
+			(hide yes)
+			(effects
+				(font
+					(size 1.27 1.27)
+				)
+			)
+		)
+		(property "MPN" "YXC X322524MMB4SI"
+			(at 137.16 137.16 0)
+			(show_name no)
+			(do_not_autoplace no)
+			(hide yes)
+			(effects
+				(font
+					(size 1.27 1.27)
+				)
 			)
 		)

Commit message: pin the passives the matcher got wrong, and close the receptacle's clearances
The fabricator's matcher put the 1 uF on a 01005 part, found nothing for the 4.7 uF or the 27 ohm,
and the ferrite's first choice ran out, so those lines carry catalogue numbers now: Samsung
CL05A105KO5NNNC and CL05A475MP5NRNC (10 V, the basic part), UNI-ROYAL 0402WGF270JTCE, Murata
BLM18KG601SN1D. The 5.1 k CC pull-downs are left to any 1 % part with stock, the specification
allowing ten percent there. The four clearances the receptacle swap left in its breakout are
closed by hand. The rules check is clean with parity and the fab files are regenerated.

Co-Authored-By: Claude Fable 5.1 <noreply@anthropic.com>
Parts:
- R15, R17: LCSC (none) -> C25100; MPN (none) -> UNI-ROYAL 0402WGF270JTCE
Changed lines of the file:
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@@
+			)
+		)
+		(property "LCSC" "C25100"
+			(at 160.02 105.41 90)
+			(show_name no)
+			(do_not_autoplace no)
+			(hide yes)
+			(effects
+				(font
+					(size 1.27 1.27)
+				)
+			)
+		)
+		(property "MPN" "UNI-ROYAL 0402WGF270JTCE"
+			(at 160.02 105.41 90)
+			(show_name no)
+			(do_not_autoplace no)
+			(hide yes)
+			(effects
+				(font
+					(size 1.27 1.27)
+				)
 			)
 		)
@@
 			(effects
 				(font
+					(size 1.27 1.27)
+				)
+			)
+		)
+		(property "LCSC" "C25100"
+			(at 152.4 107.95 90)
+			(show_name no)
+			(do_not_autoplace no)
+			(hide yes)
+			(effects
+				(font
+					(size 1.27 1.27)
+				)
+			)
+		)
+		(property "MPN" "UNI-ROYAL 0402WGF270JTCE"
+			(at 152.4 107.95 90)
+			(show_name no)
+			(do_not_autoplace no)
+			(hide yes)
+			(effects
+				(font
