File: pcb/power.kicad_sch (KiCad schematic)
At the start: 59 parts, among them J7 1S LiPo, Q1 Q_Dual_NMOS_S1G1S2G2D2D2D1D1, Q2 Q_Dual_NMOS_S1G1S2G2D2D2D1D1, Q3 Q_Dual_NMOS_S1G1S2G2D2D2D1D1, U13 BQ25798, U14 TPS63060, U15 TPS61089

Commit message: specify the resistors, and round three values that were never parts
Every resistor now carries a tolerance, and it is 1% only where the value is read: a reference a
part trims itself against, a divider ratio, a termination that states what this end of a cable is,
a value that programs a threshold at power-on. Nineteen of the thirty-eight qualify; the rest are
pull-ups, pull-downs, straps and series parts, where 5% is honest and 1% buys nothing. Power is not
a field, because the largest dissipation anywhere on the board is a few milliwatts in an
indicator's series resistor.

Three values were arithmetic nobody had rounded. 5.24k and 30.31k are the charger vendor's own
calculated figures for the temperature network and neither exists as a part; 172k was ours for the
boost's current limit and is not a standard value either. They become 5.23k, 30.1k and 174k, and
what each costs is recorded: a fraction of a degree on the temperature thresholds, about 2% on the
current limit. A fourth, the hub's reference resistor, had its tolerance written into the value
string; that moves to the field where it belongs.

Reading the boost's datasheet to round the current limit corrected how it had been described. The
limit is not set at the worst-case peak -- the switch has to pass about 4.25A at the bottom of the
cell with every port loaded, so a limit there would trip in normal service. It sits at about 5.9A,
clearing that peak by nearly 40%. The vendor publishes two resistances against measured limits,
which fixes both the relationship and its direction: more resistance, less current.

Rules check unchanged, schematic check clean.

Co-Authored-By: Claude Opus 5 (1M context) <noreply@anthropic.com>
Parts:
- R40, R41, R42, R43, R47, R48, R52: Tolerance (none) -> 5%
- R44, R49, R50, R51, R53, R54, R55: Tolerance (none) -> 1%
- R45: value 5k24 -> 5k23; Tolerance (none) -> 1%
- R46: value 30k31 -> 30k1; Tolerance (none) -> 1%
- R56: value 172k -> 174k; Tolerance (none) -> 1%
Changed lines of the file:
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@@
 			)
 		)
+		(property "Tolerance" "1%"
+			(at 307.34 167.64 0)
+			(show_name no)
+			(do_not_autoplace no)
+			(effects
+				(font
+					(size 1.27 1.27)
+				)
+				(hide yes)
+			)
+		)
 		(property "Footprint" ""
 			(at 307.34 160.02 0)
@@
 			)
 		)
+		(property "Tolerance" "5%"
+			(at 249.174 176.784 0)
+			(show_name no)
+			(do_not_autoplace no)
+			(effects
+				(font
+					(size 1.27 1.27)
+				)
+				(hide yes)
+			)
+		)
 		(property "Footprint" ""
 			(at 248.92 172.72 0)
@@
 			)
 		)
+		(property "Tolerance" "5%"
+			(at 119.38 129.54 0)
+			(show_name no)
+			(do_not_autoplace no)
+			(effects
+				(font
+					(size 1.27 1.27)
+				)
+				(hide yes)
+			)
+		)
 		(property "Footprint" ""
 			(at 119.38 121.92 0)
@@
 			)
 		)
-		(property "Value" "5k24"
+		(property "Value" "5k23"
 			(at 152.4 157.48 0)
 			(show_name no)
@@
 			)
 		)
+		(property "Tolerance" "1%"
+			(at 152.4 157.48 0)
+			(show_name no)
+			(do_not_autoplace no)
+			(effects
+				(font
+					(size 1.27 1.27)
+				)
+				(hide yes)
+			)
+		)
 		(property "Footprint" ""
 			(at 152.4 149.86 0)
@@
 			)
 		)
+		(property "Tolerance" "1%"
+			(at 292.1 102.87 0)
+			(show_name no)
+			(do_not_autoplace no)
+			(effects
+				(font
+					(size 1.27 1.27)
+				)
+				(hide yes)
+			)
+		)
 		(property "Footprint" ""
 			(at 292.1 95.25 0)
@@
 			)
 		)
+		(property "Tolerance" "1%"
+			(at 292.1 175.26 0)
+			(show_name no)
+			(do_not_autoplace no)
+			(effects
+				(font
+					(size 1.27 1.27)
+				)
+				(hide yes)
+			)
+		)
 		(property "Footprint" ""
 			(at 292.1 167.64 0)
@@
 			)
 		)
+		(property "Tolerance" "5%"
+			(at 162.56 144.78 0)
+			(show_name no)
+			(do_not_autoplace no)
+			(effects
+				(font
+					(size 1.27 1.27)
+				)
+				(hide yes)
+			)
+		)
 		(property "Footprint" ""
 			(at 162.56 137.16 0)
@@
 			)
 		)
-		(property "Value" "30k31"
+		(property "Value" "30k1"
 			(at 147.32 167.64 0)
 			(show_name no)
@@
 			)
 		)
+		(property "Tolerance" "1%"
+			(at 147.32 167.64 0)
+			(show_name no)
+			(do_not_autoplace no)
+			(effects
+				(font
+					(size 1.27 1.27)
+				)
+				(hide yes)
+			)
+		)
 		(property "Footprint" ""
 			(at 147.32 160.02 0)
@@
 			)
 		)
+		(property "Tolerance" "5%"
+			(at 195.58 137.16 0)
+			(show_name no)
+			(do_not_autoplace no)
+			(effects
+				(font
+					(size 1.27 1.27)
+				)
+				(hide yes)
+			)
+		)
 		(property "Footprint" ""
 			(at 195.58 129.54 0)
@@
 			)
 		)
+		(property "Tolerance" "5%"
+			(at 198.12 162.56 0)
+			(show_name no)
+			(do_not_autoplace no)
+			(effects
+				(font
+					(size 1.27 1.27)
+				)
+				(hide yes)
+			)
+		)
 		(property "Footprint" ""
 			(at 198.12 154.94 0)
@@
 			)
 		)
+		(property "Tolerance" "5%"
+			(at 114.3 132.08 0)
+			(show_name no)
+			(do_not_autoplace no)
+			(effects
+				(font
+					(size 1.27 1.27)
+				)
+				(hide yes)
+			)
+		)
 		(property "Footprint" ""
 			(at 114.3 124.46 0)
@@
 			)
 		)
+		(property "Tolerance" "5%"
+			(at 109.22 137.16 0)
+			(show_name no)
+			(do_not_autoplace no)
+			(effects
+				(font
+					(size 1.27 1.27)
+				)
+				(hide yes)
+			)
+		)
 		(property "Footprint" ""
 			(at 109.22 129.54 0)
@@
 			)
 		)
+		(property "Tolerance" "1%"
+			(at 246.38 170.18 0)
+			(show_name no)
+			(do_not_autoplace no)
+			(effects
+				(font
+					(size 1.27 1.27)
+				)
+				(hide yes)
+			)
+		)
 		(property "Footprint" ""
 			(at 246.38 162.56 0)
@@
 			)
 		)
-		(property "Value" "172k"
+		(property "Value" "174k"
 			(at 289.56 177.8 0)
 			(show_name no)
@@
 			)
 		)
+		(property "Tolerance" "1%"
+			(at 289.56 177.8 0)
+			(show_name no)
+			(do_not_autoplace no)
+			(effects
+				(font
+					(size 1.27 1.27)
+				)
+				(hide yes)
+			)
+		)
 		(property "Footprint" ""
 			(at 289.56 170.18 0)
@@
 			)
 		)
+		(property "Tolerance" "1%"
+			(at 307.34 176.53 0)
+			(show_name no)
+			(do_not_autoplace no)
+			(effects
+				(font
+					(size 1.27 1.27)
+				)
+				(hide yes)
+			)
+		)
 		(property "Footprint" ""
 			(at 307.34 168.91 0)
@@
 			)
 		)
+		(property "Tolerance" "1%"
+			(at 162.56 157.48 0)
+			(show_name no)
+			(do_not_autoplace no)
+			(effects
+				(font
+					(size 1.27 1.27)
+				)
+				(hide yes)
+			)
+		)
 		(property "Footprint" ""
 			(at 162.56 149.86 0)
@@
 			)
 		)
+		(property "Tolerance" "1%"
+			(at 292.1 111.76 0)
+			(show_name no)
+			(do_not_autoplace no)
+			(effects
+				(font
+					(size 1.27 1.27)
+				)
+				(hide yes)
+			)
+		)

Commit message: specify the magnetics and the crystals by what they have to do
Each inductor now states the current it has to stay unsaturated to, derived rather than copied: the
processor's own datasheet fixes 1.5A for the core regulator, the charger's output side carries
about 6.3A when the input is delivering its full 27W into a system near 4V, and each of the two
converters wants an inductor that holds up past its own current limit so the part protects itself
before the magnetics give up. The crystals state a load capacitance, which is the number that
actually decides whether they oscillate on frequency.

Two things came out of reading rather than assuming.

The charger's inductor value is not a choice. Its datasheet is explicit that 1.5MHz works only with
1uH and 750kHz only with 2.2uH, and the frequency was already fixed at power-on by the resistor
that also sets the cell count. That resistor therefore picks the inductor, and the two have to move
together or not at all. They are consistent as drawn; the coupling is now written down so they stay
that way.

The core regulator's inductor has to be fully shielded and marked for polarity, and oriented as the
vendor's layout shows, because stray field from it couples into the regulator's control loop and
moves the output even with nominally shielded parts. That is a placement constraint arriving from a
component datasheet, and it is recorded where layout will look for it rather than left in a PDF.

The processor's crystal wants a 10pF load, which the 15pF pair either side of it meets once a
couple of picofarads of stray are allowed. The hub's pair implies about 12pF by the same
arithmetic, and that one stays open: its datasheet and design checklist are both scanned images,
so nothing reads out of them without rendering the pages.

Co-Authored-By: Claude Opus 5 (1M context) <noreply@anthropic.com>
Parts:
- L10, L12: Isat (none) -> 7A; Tolerance (none) -> 20%
- L11: Isat (none) -> 3A; Tolerance (none) -> 20%
Changed lines of the file:
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@@
+			)
+		)
+		(property "Tolerance" "20%"
+			(at 207.01 121.92 0)
+			(show_name no)
+			(do_not_autoplace no)
+			(effects
+				(font
+					(size 1.27 1.27)
+				)
+				(hide yes)
+			)
+		)
+		(property "Isat" "7A"
+			(at 207.01 121.92 0)
+			(show_name no)
+			(do_not_autoplace no)
+			(effects
+				(font
+					(size 1.27 1.27)
+				)
+				(hide yes)
 			)
 		)
@@
 					(size 1.27 1.27)
 				)
+			)
+		)
+		(property "Tolerance" "20%"
+			(at 241.3 114.3 0)
+			(show_name no)
+			(do_not_autoplace no)
+			(effects
+				(font
+					(size 1.27 1.27)
+				)
+				(hide yes)
+			)
+		)
+		(property "Isat" "3A"
+			(at 241.3 114.3 0)
+			(show_name no)
+			(do_not_autoplace no)
+			(effects
+				(font
+					(size 1.27 1.27)
+				)
+				(hide yes)
 			)
 		)
@@
 			)
 		)
+		(property "Tolerance" "20%"
+			(at 243.586 160.528 0)
+			(show_name no)
+			(do_not_autoplace no)
+			(effects
+				(font
+					(size 1.27 1.27)
+				)
+				(hide yes)
+			)
+		)
+		(property "Isat" "7A"
+			(at 243.586 160.528 0)
+			(show_name no)
+			(do_not_autoplace no)
+			(effects
+				(font
+					(size 1.27 1.27)
+				)
+				(hide yes)
+			)
+		)

Commit message: take a two-wire cell, and put the thermistor on the board
The cell connector becomes two ways on 2.0mm pitch, which is what is actually sold, and the sensor
the pack does not carry goes on the board instead. The charger's temperature network is otherwise
unchanged: the same two resistors, computed by its vendor for a 10k sensor, with the thermistor now
across the lower leg exactly where the pack's would have connected. It has to be a 10k B3435 part,
because that is the sensor those resistors were calculated against.

What the protection means changes, and the document now says so rather than leaving the impression
intact. A thermistor in the pack watches the cell; one on the board watches the board. It can no
longer catch a cell heating up by itself, which is the failure people picture when they think of
battery thermal protection. What it does instead is refuse to charge when the surroundings are too
cold or too hot for charging to be safe -- which is worth having, since charging a lithium cell
below freezing damages it permanently and ambient is a fair proxy for a resting cell. It is a
different guarantee, and the specification should state which one the product makes.

It also turns a component into a placement requirement: the sensor sits against the cell and away
from the charger, the converters and their inductors. Near a heat source it reads high and refuses
to charge a good cell; out in open board it reads ambient and says nothing about the battery. The
first of those will be blamed on firmware.

Connection list reads as expected -- the sensor, both divider legs and the charger's sense pin on
one node, the cell's return and the sensor's other end on ground.

Co-Authored-By: Claude Opus 5 (1M context) <noreply@anthropic.com>
Parts:
- removed J7: 1S LiPo, symbol Connector_Generic:Conn_01x03
- added J7: 1S LiPo, symbol Connector_Generic:Conn_01x02
- added TH1: 10k B3435, symbol Device:Thermistor_NTC
Connections:
- net BATT: now also J7.1 (Pin_1)
- net GND: now also J7.2 (Pin_2), TH1.2
- net NTC: now also TH1.1
Changed lines of the file:
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@@
 	(wire
 		(pts
-			(xy 147.32 208.28) (xy 142.24 208.28)
-		)
-		(stroke
-			(width 0)
-			(type solid)
-		)
-	)
-	(wire
-		(pts
 			(xy 276.86 91.44) (xy 304.8 91.44)
 		)
@@
 	(wire
 		(pts
-			(xy 147.32 205.74) (xy 134.62 205.74)
-		)
-		(stroke
-			(width 0)
-			(type solid)
-		)
-	)
-	(wire
-		(pts
 			(xy 276.86 106.68) (xy 289.56 106.68)
 		)
@@
 		)
 	)
-	(label "NTC"
-		(at 134.62 205.74 0)
-		(effects
-			(font
-				(size 1.27 1.27)
-			)
-			(justify left bottom)
-		)
-	)
 	(label "VSYS"
 		(at 48.26 157.48 0)
@@
 	)
 	(symbol
-		(lib_id "Connector_Generic:Conn_01x03")
-		(at 152.4 205.74 0)
-		(unit 1)
-		(body_style 1)
-		(exclude_from_sim no)
-		(in_bom yes)
-		(on_board yes)
-		(in_pos_files yes)
-		(dnp no)
-		(property "Reference" "J7"
-			(at 152.4 198.12 0)
-			(show_name no)
-			(do_not_autoplace no)
-			(effects
-				(font
-					(size 1.27 1.27)
-				)
-			)
-		)
-		(property "Value" "1S LiPo"
-			(at 152.4 213.36 0)
-			(show_name no)
-			(do_not_autoplace no)
-			(effects
-				(font
-					(size 1.27 1.27)
-				)
-			)
-		)
-		(property "Footprint" ""
-			(at 152.4 205.74 0)
-			(show_name no)
-			(do_not_autoplace no)
-			(effects
-				(font
-					(size 1.27 1.27)
-				)
-			)
-		)
-		(property "Datasheet" ""
-			(at 152.4 205.74 0)
-			(show_name no)
-			(do_not_autoplace no)
-			(effects
-				(font
-					(size 1.27 1.27)
-				)
-			)
-		)
-		(property "Description" ""
-			(at 152.4 205.74 0)
-			(show_name no)
-			(do_not_autoplace no)
-			(effects
-				(font
-					(size 1.27 1.27)
-				)
-			)
-		)
-		(pin "1"
-		)
-		(pin "2"
-		)
-		(pin "3"
-		)
-		(instances
-			(project "crossfire"
-				(path "/4c5cdd13-4f54-43b0-affb-0ae4b9a4d279/3a0d800d-f868-47e5-a520-4703480651cc"
-					(reference "J7")
-					(unit 1)
-				)
-			)
-		)
-	)
-	(symbol
 		(lib_id "power:PWR_FLAG")
 		(at 118.11 77.47 0)
@@
 		(diameter 0)
 		(color 0 0 0 0)
+	)
+	(symbol
+		(lib_id "Connector_Generic:Conn_01x02")
+		(at 152.40 203.20 0)
+		(unit 1)
+		(body_style 1)
+		(exclude_from_sim no)
+		(in_bom yes)
+		(on_board yes)
+		(in_pos_files yes)
+		(dnp no)
+		(property "Reference" "J7"
+			(at 152.40 195.58 0)
+			(show_name no)
+			(do_not_autoplace no)
+			(effects
+				(font
+					(size 1.27 1.27)
+				)
+				(justify left)
+			)
+		)
+		(property "Value" "1S LiPo"
+			(at 152.40 213.36 0)
+			(show_name no)
+			(do_not_autoplace no)
+			(effects
+				(font
+					(size 1.27 1.27)
+				)
+				(justify left)
+			)
+		)
+		(property "Footprint" ""
+			(at 152.40 203.20 0)
+			(show_name no)
+			(do_not_autoplace no)
+			(effects
+				(font
+					(size 1.27 1.27)
+				)
+				(hide yes)
+			)
+		)
+		(property "Datasheet" ""
+			(at 152.40 203.20 0)
+			(show_name no)
+			(do_not_autoplace no)
+			(effects
+				(font
+					(size 1.27 1.27)
+				)
+				(hide yes)
+			)
+		)
+		(property "Description" ""
+			(at 152.40 203.20 0)
+			(show_name no)
+			(do_not_autoplace no)
+			(effects
+				(font
+					(size 1.27 1.27)
+				)
+				(hide yes)
+			)
+		)
+		(pin "1"
+		)
+		(pin "2"
+		)
+		(instances
+			(project "crossfire"
+				(path "/4c5cdd13-4f54-43b0-affb-0ae4b9a4d279/3a0d800d-f868-47e5-a520-4703480651cc"
+					(reference "J7")
+					(unit 1)
+				)
+			)
+		)
+	)
+	(wire
+		(pts
+			(xy 147.32 205.74) (xy 142.24 205.74)
+		)
+		(stroke
+			(width 0)
+			(type default)
+		)
+	)
+	(wire
+		(pts
+			(xy 142.24 205.74) (xy 142.24 208.28)
+		)
+		(stroke
+			(width 0)
+			(type default)
+		)
+	)
+	(symbol
+		(lib_id "Device:Thermistor_NTC")
+		(at 142.24 161.29 0)
+		(unit 1)
+		(body_style 1)
+		(exclude_from_sim no)
+		(in_bom yes)
+		(on_board yes)
+		(in_pos_files yes)
+		(dnp no)
+		(property "Reference" "TH1"
+			(at 142.24 134.62 0)
+			(show_name no)
+			(do_not_autoplace no)
+			(effects
+				(font
+					(size 1.27 1.27)
+				)
+				(justify left)
+			)
+		)
+		(property "Value" "10k B3435"
+			(at 142.24 166.37 0)
+			(show_name no)
+			(do_not_autoplace no)
+			(effects
+				(font
+					(size 1.27 1.27)
+				)
+				(justify left)
+			)
+		)
+		(property "Footprint" ""
+			(at 142.24 161.29 0)
+			(show_name no)
+			(do_not_autoplace no)
+			(effects
+				(font
+					(size 1.27 1.27)
+				)
+				(hide yes)
+			)
+		)
+		(property "Datasheet" ""
+			(at 142.24 161.29 0)
+			(show_name no)
+			(do_not_autoplace no)
+			(effects
+				(font
+					(size 1.27 1.27)
+				)
+				(hide yes)
+			)
+		)
+		(property "Description" ""
+			(at 142.24 161.29 0)
+			(show_name no)
+			(do_not_autoplace no)
+			(effects
+				(font
+					(size 1.27 1.27)
+				)
+				(hide yes)
+			)
+		)
+		(pin "1"
+		)
+		(pin "2"
+		)
+		(instances
+			(project "crossfire"
+				(path "/4c5cdd13-4f54-43b0-affb-0ae4b9a4d279/3a0d800d-f868-47e5-a520-4703480651cc"
+					(reference "TH1")
+					(unit 1)
+				)
+			)
+		)
+	)
+	(wire
+		(pts
+			(xy 142.24 154.94) (xy 142.24 157.48)
+		)
+		(stroke
+			(width 0)
+			(type default)
+		)
+	)
+	(wire
+		(pts
+			(xy 142.24 165.10) (xy 147.32 165.10)
+		)
+		(stroke
+			(width 0)
+			(type default)
+		)
+	)
+	(junction
+		(at 147.32 165.10)
+		(diameter 0)
+		(color 0 0 0 0)
