File: pcb/power.kicad_sch (KiCad schematic)
At the start: 11 parts, among them U4 AP63203WU

Commit message: settle the open items by reading, pick the fabricator, and script the export
The flash is rated 133 MHz for everything but the plain read, so the QSPI divider's 120 MHz
stands. The buck's values are checked against its datasheet's table and text: the 4.7 uH stays
inside the recommended band with 0.22 A of ripple; the input capacitor becomes the same 10 uF 0805
16 V X7R part as the hub's bulk capacitor, so it still reads 10 uF with 5 V across it; the inductor
is named, a Coilcraft XEL4030-472MEC on the land already placed, chosen over the XFL part in the
same size because that one saturates below the buck's current limit. VBUS carries 10.6 uF nominal
and about 8 uF real at attach, under the 10 uF allowed. The three items that only a prototype can
answer move to their own list, with the crystals' drive level added to it.

The board goes to JLCPCB assembled: four layers with 0.2 mm vias is its standard process, it fills
and caps vias in pads, it assembles both faces and through-hole, and the four chips that matter
are in its catalogue -- their numbers are now LCSC fields on the symbols and a column in the bill
of materials. The two connectors are not, and go in as sourced or consigned parts.

scripts/export-fab.ps1 writes the Gerber and drill zip, the bill of materials and the placement
file to pcb/fab/ (untracked), after a rules check with schematic parity that refills the pours and
saves the board first, since the Gerbers are plotted from the stored fill. The first run found the
fill a step behind the last edit, which the saved board now carries.

The board still has the old C20 footprint and lacks the new fields until the schematic is pushed
to it, which is the next step before the export passes.

Co-Authored-By: Claude Fable 5.1 <noreply@anthropic.com>
Parts:
- C20: footprint Capacitor_SMD:C_0603_1608Metric -> Capacitor_SMD:C_0805_2012Metric; Dielectric X5R -> X7R; Voltage 10V -> 16V
- L2: DCR (none) -> 44mR max; Isat 2A min -> 4.6A; MPN 4.7 uH, 4 mm shielded; part to confirm -> Coilcraft XEL4030-472MEC
- U4: LCSC (none) -> C780769; MPN (none) -> AP63203WU-7
Changed lines of the file:
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@@
+			)
+		)
+		(property "DCR" "44mR max"
+			(at 177.8 96.52 90)
+			(show_name no)
+			(do_not_autoplace no)
+			(hide yes)
+			(effects
+				(font
+					(size 1.27 1.27)
+				)
+				(justify left)
 			)
 		)
@@
 			)
 		)
-		(property "MPN" "4.7 uH, 4 mm shielded; part to confirm"
+		(property "MPN" "Coilcraft XEL4030-472MEC"
 			(at 177.8 106.68 0)
 			(hide yes)
@@
 			)
 		)
-		(property "Isat" "2A min"
+		(property "Isat" "4.6A"
 			(at 177.8 106.68 0)
 			(hide yes)
@@
 			)
 		)
-		(property "Footprint" "Capacitor_SMD:C_0603_1608Metric"
+		(property "Footprint" "Capacitor_SMD:C_0805_2012Metric"
 			(at 116.84 101.6 0)
 			(hide yes)
@@
 			)
 		)
-		(property "Voltage" "10V"
+		(property "Voltage" "16V"
 			(at 116.84 109.22 0)
 			(hide yes)
@@
 			)
 		)
-		(property "Dielectric" "X5R"
+		(property "Dielectric" "X7R"
 			(at 116.84 109.22 0)
 			(hide yes)
@@
 			(effects
 				(font
+					(size 1.27 1.27)
+				)
+			)
+		)
+		(property "MPN" "AP63203WU-7"
+			(at 156.21 93.98 0)
+			(show_name no)
+			(do_not_autoplace no)
+			(hide yes)
+			(effects
+				(font
+					(size 1.27 1.27)
+				)
+			)
+		)
+		(property "LCSC" "C780769"
+			(at 156.21 93.98 0)
+			(show_name no)
+			(do_not_autoplace no)
+			(hide yes)
+			(effects
+				(font

Commit message: every bill-of-materials line answers the assembler
The first upload to the fabricator matched the passives by value and package and failed nine
lines. Each line now carries a definite answer in the schematic, written out as columns: a
catalogue number where the part is in the catalogue -- the flash, the protection arrays, the
indicators, the ferrite, and both crystals as 10 pF parts, since the catalogue's basic crystals
are 20 pF and the processor vendor's circuit was copied with its 15 pF capacitors; a named part
and a global-sourcing note where it is not -- the buck inductor, the buttons, the USB-C receptacle
and the USB-A sockets. The debug header is marked not fitted, and the mounting holes leave the
bill and the placement file, since neither is a part.

The same fields are on the board's footprints, as an update from the schematic would put them, so
parity holds; the export writes the sourcing column; the design document carries the table.

Co-Authored-By: Claude Fable 5.1 <noreply@anthropic.com>
Parts:
- L2: Sourcing (none) -> JLCPCB global sourcing
Changed lines of the file:
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@@
+			)
+		)
+		(property "Sourcing" "JLCPCB global sourcing"
+			(at 177.8 96.52 90)
+			(show_name no)
+			(do_not_autoplace no)
+			(hide yes)
+			(effects
+				(font
+					(size 1.27 1.27)
+				)
+				(justify left)
 			)
 		)
