File: pcb/port.kicad_sch (KiCad schematic)
At the start: 4 parts, among them J2 USB_A, U4 TPS2065C, U5 USBLC6-2SC6

Commit message: checkpoint the battery, PD and radio design as it stood
The last state of the full-featured board before it is reduced to a single
USB-C input: the power block re-placed part by part in order of importance,
the charger's signal pins fanned out, the differential pairs renamed so the
layout tool recognises them, the 3.3 V converter's feedback divider joined
to its pin, the FETs given their part number, and the non-printing fields
hidden on the schematic. The layout is incomplete and is recorded as such.

Co-Authored-By: Claude Fable 5.1 <noreply@anthropic.com>
Connections:
- net CONN_D-: now reaches J2.2 (D-), U5.4 (I/O2)
- net CONN_D+: now reaches J2.3 (D+), U5.6 (I/O1)
- net DM renamed D-
- net DP renamed D+
Changed lines of the file:
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@@
+		)
+	)
+	(label "CONN_D-"
+		(at 172.72 111.76 0)
+		(effects
+			(font
+				(size 1.27 1.27)
+			)
+			(justify left bottom)
+		)
+	)
+	(label "CONN_D+"
+		(at 172.72 109.22 0)
+		(effects
+			(font
+				(size 1.27 1.27)
+			)
+			(justify left bottom)
 		)
 	)
@@
 		)
 	)
-	(hierarchical_label "DP"
+	(hierarchical_label "D+"
 		(shape bidirectional)
 		(at 139.7 109.22 180)
@@
 		)
 	)
-	(hierarchical_label "DM"
+	(hierarchical_label "D-"
 		(shape bidirectional)
 		(at 139.7 111.76 180)
@@
 		(in_pos_files yes)
 		(dnp no)
-		(property "Reference" "#PWR042"
+		(property "Reference" "#PWR044"
 			(at 173.99 80.01 0)
 			(hide yes)
@@
 		(property "Footprint" ""
 			(at 173.99 87.63 0)
+			(hide yes)
 			(show_name no)
 			(do_not_autoplace no)
@@
 		(property "Datasheet" ""
 			(at 173.99 87.63 0)
+			(hide yes)
 			(show_name no)
 			(do_not_autoplace no)
@@
 		(property "Description" ""
 			(at 173.99 87.63 0)
+			(hide yes)
 			(show_name no)
 			(do_not_autoplace no)
@@
 		(property "Footprint" "Package_TO_SOT_SMD:SOT-23-6"
 			(at 160.02 109.22 0)
+			(hide yes)
 			(show_name no)
 			(do_not_autoplace no)
@@
 		(property "Datasheet" ""
 			(at 160.02 109.22 0)
+			(hide yes)
 			(show_name no)
 			(do_not_autoplace no)
@@
 		(property "Description" ""
 			(at 160.02 109.22 0)
+			(hide yes)
 			(show_name no)
 			(do_not_autoplace no)
@@
 		(in_pos_files yes)
 		(dnp no)
-		(property "Reference" "#PWR046"
+		(property "Reference" "#PWR048"
 			(at 196.85 116.84 0)
 			(hide yes)
@@
 		(property "Footprint" ""
 			(at 196.85 124.46 0)
+			(hide yes)
 			(show_name no)
 			(do_not_autoplace no)
@@
 		(property "Datasheet" ""
 			(at 196.85 124.46 0)
+			(hide yes)
 			(show_name no)
 			(do_not_autoplace no)
@@
 		(property "Description" ""
 			(at 196.85 124.46 0)
+			(hide yes)
 			(show_name no)
 			(do_not_autoplace no)
@@
 		(in_pos_files yes)
 		(dnp no)
-		(property "Reference" "#PWR050"
+		(property "Reference" "#PWR052"
 			(at 111.76 88.9 0)
 			(hide yes)
@@
 		(property "Footprint" ""
 			(at 111.76 96.52 0)
+			(hide yes)
 			(show_name no)
 			(do_not_autoplace no)
@@
 		(property "Datasheet" ""
 			(at 111.76 96.52 0)
+			(hide yes)
 			(show_name no)
 			(do_not_autoplace no)
@@
 		(property "Description" ""
 			(at 111.76 96.52 0)
+			(hide yes)
 			(show_name no)
 			(do_not_autoplace no)
@@
 		(property "Footprint" "Connector_USB:USB_A_Molex_67643_Horizontal"
 			(at 190.5 109.22 0)
+			(hide yes)
 			(show_name no)
 			(do_not_autoplace no)
@@
 		(property "Datasheet" ""
 			(at 190.5 109.22 0)
+			(hide yes)
 			(show_name no)
 			(do_not_autoplace no)
@@
 		(property "Description" ""
 			(at 190.5 109.22 0)
+			(hide yes)
 			(show_name no)
 			(do_not_autoplace no)
@@
 			)
 		)
+		(property "Footprint" "Capacitor_SMD:C_1210_3225Metric"
+			(at 168.91 91.44 0)
+			(hide yes)
+			(show_name no)
+			(do_not_autoplace no)
+			(effects
+				(font
+					(size 1.27 1.27)
+				)
+			)
+		)
+		(property "Datasheet" ""
+			(at 168.91 91.44 0)
+			(hide yes)
+			(show_name no)
+			(do_not_autoplace no)
+			(effects
+				(font
+					(size 1.27 1.27)
+				)
+			)
+		)
+		(property "Description" ""
+			(at 168.91 91.44 0)
+			(hide yes)
+			(show_name no)
+			(do_not_autoplace no)
+			(effects
+				(font
+					(size 1.27 1.27)
+				)
+			)
+		)
 		(property "Voltage" "25V"
 			(at 171.958 93.726 0)
-			(show_name no)
-			(do_not_autoplace no)
-			(effects
-				(font
-					(size 1.27 1.27)
-				)
-				(hide yes)
+			(hide yes)
+			(show_name no)
+			(do_not_autoplace no)
+			(effects
+				(font
+					(size 1.27 1.27)
+				)
 			)
 		)
 		(property "Dielectric" "X7R"
 			(at 171.958 93.726 0)
-			(show_name no)
-			(do_not_autoplace no)
-			(effects
-				(font
-					(size 1.27 1.27)
-				)
-				(hide yes)
-			)
-		)
-		(property "Footprint" "Capacitor_SMD:C_1210_3225Metric"
-			(at 168.91 91.44 0)
-			(show_name no)
-			(do_not_autoplace no)
-			(effects
-				(font
-					(size 1.27 1.27)
-				)
-			)
-		)
-		(property "Datasheet" ""
-			(at 168.91 91.44 0)
-			(show_name no)
-			(do_not_autoplace no)
-			(effects
-				(font
-					(size 1.27 1.27)
-				)
-			)
-		)
-		(property "Description" ""
-			(at 168.91 91.44 0)
+			(hide yes)
 			(show_name no)
 			(do_not_autoplace no)
@@
 		(property "Footprint" "Package_TO_SOT_SMD:SOT-23-5"
 			(at 127 99.06 0)
+			(hide yes)
 			(show_name no)
 			(do_not_autoplace no)
@@
 		(property "Datasheet" ""
 			(at 127 99.06 0)
+			(hide yes)
 			(show_name no)
 			(do_not_autoplace no)
@@
 		(property "Description" ""
 			(at 127 99.06 0)
-			(show_name no)
-			(do_not_autoplace no)
+			(hide yes)
+			(show_name no)
+			(do_not_autoplace no)
