File: pcb/port.kicad_sch (KiCad schematic)
At the start: 4 parts, among them J2 USB_A, U4 TPS2065C, U5 USBLC6-2SC6

Commit message: manual pcb finishing work
Parts:
- renumbered C40 to C39, J2 to J3, U4 to U6, U5 to U7
Changed lines of the file:
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@@
 		(in_pos_files yes)
 		(dnp no)
-		(property "Reference" "#PWR044"
+		(property "Reference" "#PWR072"
 			(at 173.99 80.01 0)
 			(hide yes)
@@
 			(project "crossfire"
 				(path "/4c5cdd13-4f54-43b0-affb-0ae4b9a4d279/1ec2d2db-5a93-44dc-ab43-bd5c3109edb6"
-					(reference "#PWR042")
+					(reference "#PWR081")
 					(unit 1)
 				)
 				(path "/4c5cdd13-4f54-43b0-affb-0ae4b9a4d279/5d450cbf-9176-48a8-abac-f4efc13cd215"
-					(reference "#PWR043")
+					(reference "#PWR078")
 					(unit 1)
 				)
 				(path "/4c5cdd13-4f54-43b0-affb-0ae4b9a4d279/970bba49-0501-4f56-a5bb-beb1a684622b"
-					(reference "#PWR044")
+					(reference "#PWR072")
 					(unit 1)
 				)
 				(path "/4c5cdd13-4f54-43b0-affb-0ae4b9a4d279/e01ae319-731b-4a6e-aad5-fb5dc353047a"
-					(reference "#PWR045")
+					(reference "#PWR075")
 					(unit 1)
 				)
@@
 		(in_pos_files yes)
 		(dnp no)
-		(property "Reference" "U5"
+		(property "Reference" "U7"
 			(at 160.02 101.6 0)
 			(show_name no)
@@
 			(project "crossfire"
 				(path "/4c5cdd13-4f54-43b0-affb-0ae4b9a4d279/1ec2d2db-5a93-44dc-ab43-bd5c3109edb6"
+					(reference "U13")
+					(unit 1)
+				)
+				(path "/4c5cdd13-4f54-43b0-affb-0ae4b9a4d279/5d450cbf-9176-48a8-abac-f4efc13cd215"
 					(reference "U11")
 					(unit 1)
 				)
-				(path "/4c5cdd13-4f54-43b0-affb-0ae4b9a4d279/5d450cbf-9176-48a8-abac-f4efc13cd215"
+				(path "/4c5cdd13-4f54-43b0-affb-0ae4b9a4d279/970bba49-0501-4f56-a5bb-beb1a684622b"
+					(reference "U7")
+					(unit 1)
+				)
+				(path "/4c5cdd13-4f54-43b0-affb-0ae4b9a4d279/e01ae319-731b-4a6e-aad5-fb5dc353047a"
 					(reference "U9")
-					(unit 1)
-				)
-				(path "/4c5cdd13-4f54-43b0-affb-0ae4b9a4d279/970bba49-0501-4f56-a5bb-beb1a684622b"
-					(reference "U5")
-					(unit 1)
-				)
-				(path "/4c5cdd13-4f54-43b0-affb-0ae4b9a4d279/e01ae319-731b-4a6e-aad5-fb5dc353047a"
-					(reference "U7")
 					(unit 1)
 				)
@@
 		(in_pos_files yes)
 		(dnp no)
-		(property "Reference" "#PWR048"
+		(property "Reference" "#PWR073"
 			(at 196.85 116.84 0)
 			(hide yes)
@@
 			(project "crossfire"
 				(path "/4c5cdd13-4f54-43b0-affb-0ae4b9a4d279/1ec2d2db-5a93-44dc-ab43-bd5c3109edb6"
-					(reference "#PWR046")
+					(reference "#PWR082")
 					(unit 1)
 				)
 				(path "/4c5cdd13-4f54-43b0-affb-0ae4b9a4d279/5d450cbf-9176-48a8-abac-f4efc13cd215"
-					(reference "#PWR047")
+					(reference "#PWR079")
 					(unit 1)
 				)
 				(path "/4c5cdd13-4f54-43b0-affb-0ae4b9a4d279/970bba49-0501-4f56-a5bb-beb1a684622b"
-					(reference "#PWR048")
+					(reference "#PWR073")
 					(unit 1)
 				)
 				(path "/4c5cdd13-4f54-43b0-affb-0ae4b9a4d279/e01ae319-731b-4a6e-aad5-fb5dc353047a"
-					(reference "#PWR049")
+					(reference "#PWR076")
 					(unit 1)
 				)
@@
 		(in_pos_files yes)
 		(dnp no)
-		(property "Reference" "#PWR052"
+		(property "Reference" "#PWR071"
 			(at 111.76 88.9 0)
 			(hide yes)
@@
 			(project "crossfire"
 				(path "/4c5cdd13-4f54-43b0-affb-0ae4b9a4d279/1ec2d2db-5a93-44dc-ab43-bd5c3109edb6"
-					(reference "#PWR050")
+					(reference "#PWR080")
 					(unit 1)
 				)
 				(path "/4c5cdd13-4f54-43b0-affb-0ae4b9a4d279/5d450cbf-9176-48a8-abac-f4efc13cd215"
-					(reference "#PWR051")
+					(reference "#PWR077")
 					(unit 1)
 				)
 				(path "/4c5cdd13-4f54-43b0-affb-0ae4b9a4d279/970bba49-0501-4f56-a5bb-beb1a684622b"
-					(reference "#PWR052")
+					(reference "#PWR071")
 					(unit 1)
 				)
 				(path "/4c5cdd13-4f54-43b0-affb-0ae4b9a4d279/e01ae319-731b-4a6e-aad5-fb5dc353047a"
-					(reference "#PWR053")
+					(reference "#PWR074")
 					(unit 1)
 				)
@@
 		(in_pos_files yes)
 		(dnp no)
-		(property "Reference" "J2"
+		(property "Reference" "J3"
 			(at 190.5 101.6 0)
 			(show_name no)
@@
 			(project "crossfire"
 				(path "/4c5cdd13-4f54-43b0-affb-0ae4b9a4d279/1ec2d2db-5a93-44dc-ab43-bd5c3109edb6"
+					(reference "J6")
+					(unit 1)
+				)
+				(path "/4c5cdd13-4f54-43b0-affb-0ae4b9a4d279/5d450cbf-9176-48a8-abac-f4efc13cd215"
 					(reference "J5")
 					(unit 1)
 				)
-				(path "/4c5cdd13-4f54-43b0-affb-0ae4b9a4d279/5d450cbf-9176-48a8-abac-f4efc13cd215"
+				(path "/4c5cdd13-4f54-43b0-affb-0ae4b9a4d279/970bba49-0501-4f56-a5bb-beb1a684622b"
+					(reference "J3")
+					(unit 1)
+				)
+				(path "/4c5cdd13-4f54-43b0-affb-0ae4b9a4d279/e01ae319-731b-4a6e-aad5-fb5dc353047a"
 					(reference "J4")
-					(unit 1)
-				)
-				(path "/4c5cdd13-4f54-43b0-affb-0ae4b9a4d279/970bba49-0501-4f56-a5bb-beb1a684622b"
-					(reference "J2")
-					(unit 1)
-				)
-				(path "/4c5cdd13-4f54-43b0-affb-0ae4b9a4d279/e01ae319-731b-4a6e-aad5-fb5dc353047a"
-					(reference "J3")
 					(unit 1)
 				)
@@
 		(in_pos_files yes)
 		(dnp no)
-		(property "Reference" "C40"
+		(property "Reference" "C39"
 			(at 166.37 89.408 0)
 			(show_name no)
@@
 			(project "crossfire"
 				(path "/4c5cdd13-4f54-43b0-affb-0ae4b9a4d279/1ec2d2db-5a93-44dc-ab43-bd5c3109edb6"
-					(reference "C43")
+					(reference "C42")
 					(unit 1)
 				)
 				(path "/4c5cdd13-4f54-43b0-affb-0ae4b9a4d279/5d450cbf-9176-48a8-abac-f4efc13cd215"
-					(reference "C42")
+					(reference "C41")
 					(unit 1)
 				)
 				(path "/4c5cdd13-4f54-43b0-affb-0ae4b9a4d279/970bba49-0501-4f56-a5bb-beb1a684622b"
+					(reference "C39")
+					(unit 1)
+				)
+				(path "/4c5cdd13-4f54-43b0-affb-0ae4b9a4d279/e01ae319-731b-4a6e-aad5-fb5dc353047a"
 					(reference "C40")
-					(unit 1)
-				)
-				(path "/4c5cdd13-4f54-43b0-affb-0ae4b9a4d279/e01ae319-731b-4a6e-aad5-fb5dc353047a"
-					(reference "C41")
 					(unit 1)
 				)
@@
 		(in_pos_files yes)
 		(dnp no)
-		(property "Reference" "U4"
+		(property "Reference" "U6"
 			(at 127 91.44 0)
 			(show_name no)
@@
 			(project "crossfire"
 				(path "/4c5cdd13-4f54-43b0-affb-0ae4b9a4d279/1ec2d2db-5a93-44dc-ab43-bd5c3109edb6"
+					(reference "U12")
+					(unit 1)
+				)
+				(path "/4c5cdd13-4f54-43b0-affb-0ae4b9a4d279/5d450cbf-9176-48a8-abac-f4efc13cd215"
 					(reference "U10")
 					(unit 1)
 				)
-				(path "/4c5cdd13-4f54-43b0-affb-0ae4b9a4d279/5d450cbf-9176-48a8-abac-f4efc13cd215"
+				(path "/4c5cdd13-4f54-43b0-affb-0ae4b9a4d279/970bba49-0501-4f56-a5bb-beb1a684622b"
+					(reference "U6")
+					(unit 1)
+				)
+				(path "/4c5cdd13-4f54-43b0-affb-0ae4b9a4d279/e01ae319-731b-4a6e-aad5-fb5dc353047a"
 					(reference "U8")
 					(unit 1)
 				)
-				(path "/4c5cdd13-4f54-43b0-affb-0ae4b9a4d279/970bba49-0501-4f56-a5bb-beb1a684622b"
-					(reference "U4")
-					(unit 1)
-				)
-				(path "/4c5cdd13-4f54-43b0-affb-0ae4b9a4d279/e01ae319-731b-4a6e-aad5-fb5dc353047a"
-					(reference "U6")
-					(unit 1)
-				)
