File: pcb/port.kicad_sch (KiCad schematic)
At the start: 4 parts, among them J3 USB_A, U6 TPS2065C, U7 USBLC6-2SC6

Commit message: cut the front edge at the sockets' edge marking
The receptacle footprint marks on its fabrication layer where the board edge belongs, 3.7 mm
behind the socket face, and the outline was cut flush with the face instead. With every part now
placed behind the marking, the front edge moves up to it: the board is 100 x 49.78 mm, the bottom
corners keep their radius, each pour keeps its inset from the edge, and the row of stitching vias
that stood in the strip is gone. The front mounting hole on the right is set level with the one on
the left, which is the clearance it needed from the new edge.

The sockets take a project copy of the library footprint whose silkscreen stops inside the edge
marking, since the library's draws the whole body and every line of it that crossed the edge was
reported. Pads, courtyard and fabrication drawing are the library's; the port sheet names the copy.

Co-Authored-By: Claude Fable 5.1 <noreply@anthropic.com>
Parts:
- J3: footprint Connector_USB:USB_A_Molex_67643_Horizontal -> crossfire:USB_A_Molex_67643_Horizontal_Overhang
Changed lines of the file:
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@@
 			)
 		)
-		(property "Footprint" "Connector_USB:USB_A_Molex_67643_Horizontal"
+		(property "Footprint" "crossfire:USB_A_Molex_67643_Horizontal_Overhang"
 			(at 190.5 109.22 0)
 			(hide yes)

Commit message: settle the open items by reading, pick the fabricator, and script the export
The flash is rated 133 MHz for everything but the plain read, so the QSPI divider's 120 MHz
stands. The buck's values are checked against its datasheet's table and text: the 4.7 uH stays
inside the recommended band with 0.22 A of ripple; the input capacitor becomes the same 10 uF 0805
16 V X7R part as the hub's bulk capacitor, so it still reads 10 uF with 5 V across it; the inductor
is named, a Coilcraft XEL4030-472MEC on the land already placed, chosen over the XFL part in the
same size because that one saturates below the buck's current limit. VBUS carries 10.6 uF nominal
and about 8 uF real at attach, under the 10 uF allowed. The three items that only a prototype can
answer move to their own list, with the crystals' drive level added to it.

The board goes to JLCPCB assembled: four layers with 0.2 mm vias is its standard process, it fills
and caps vias in pads, it assembles both faces and through-hole, and the four chips that matter
are in its catalogue -- their numbers are now LCSC fields on the symbols and a column in the bill
of materials. The two connectors are not, and go in as sourced or consigned parts.

scripts/export-fab.ps1 writes the Gerber and drill zip, the bill of materials and the placement
file to pcb/fab/ (untracked), after a rules check with schematic parity that refills the pours and
saves the board first, since the Gerbers are plotted from the stored fill. The first run found the
fill a step behind the last edit, which the saved board now carries.

The board still has the old C20 footprint and lacks the new fields until the schematic is pushed
to it, which is the next step before the export passes.

Co-Authored-By: Claude Fable 5.1 <noreply@anthropic.com>
Parts:
- U6: LCSC (none) -> C353882; MPN (none) -> TPS2065CDBVR
Changed lines of the file:
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@@
+			)
+		)
+		(property "MPN" "TPS2065CDBVR"
+			(at 127 106.68 0)
+			(show_name no)
+			(do_not_autoplace no)
+			(hide yes)
+			(effects
+				(font
+					(size 1.27 1.27)
+				)
+			)
+		)
+		(property "LCSC" "C353882"
+			(at 127 106.68 0)
+			(show_name no)
+			(do_not_autoplace no)
+			(hide yes)
+			(effects
+				(font
+					(size 1.27 1.27)
+				)
 			)
 		)

Commit message: every bill-of-materials line answers the assembler
The first upload to the fabricator matched the passives by value and package and failed nine
lines. Each line now carries a definite answer in the schematic, written out as columns: a
catalogue number where the part is in the catalogue -- the flash, the protection arrays, the
indicators, the ferrite, and both crystals as 10 pF parts, since the catalogue's basic crystals
are 20 pF and the processor vendor's circuit was copied with its 15 pF capacitors; a named part
and a global-sourcing note where it is not -- the buck inductor, the buttons, the USB-C receptacle
and the USB-A sockets. The debug header is marked not fitted, and the mounting holes leave the
bill and the placement file, since neither is a part.

The same fields are on the board's footprints, as an update from the schematic would put them, so
parity holds; the export writes the sourcing column; the design document carries the table.

Co-Authored-By: Claude Fable 5.1 <noreply@anthropic.com>
Parts:
- J3: MPN (none) -> Molex 0676430910; Sourcing (none) -> JLCPCB global sourcing
- U7: LCSC (none) -> C7519; MPN (none) -> USBLC6-2SC6
Changed lines of the file:
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@@
+			)
+		)
+		(property "LCSC" "C7519"
+			(at 160.02 116.84 0)
+			(show_name no)
+			(do_not_autoplace no)
+			(hide yes)
+			(effects
+				(font
+					(size 1.27 1.27)
+				)
+			)
+		)
+		(property "MPN" "USBLC6-2SC6"
+			(at 160.02 116.84 0)
+			(show_name no)
+			(do_not_autoplace no)
+			(hide yes)
+			(effects
+				(font
+					(size 1.27 1.27)
+				)
 			)
 		)
@@
 			(effects
 				(font
+					(size 1.27 1.27)
+				)
+			)
+		)
+		(property "Sourcing" "JLCPCB global sourcing"
+			(at 190.5 116.84 0)
+			(show_name no)
+			(do_not_autoplace no)
+			(hide yes)
+			(effects
+				(font
+					(size 1.27 1.27)
+				)
+			)
+		)
+		(property "MPN" "Molex 0676430910"
+			(at 190.5 116.84 0)
+			(show_name no)
+			(do_not_autoplace no)
+			(hide yes)
+			(effects
+				(font

Commit message: the four sourced lines become catalogue parts
Global sourcing turned out to be a pre-purchase into one's own library, three to four weeks and an
inspection fee per kind of connector or switch, so the connectors, the buttons and the prototype's
inductor come from the catalogue instead, each checked against a drawing rather than a part page:

- USB-C: Korean Hroparts TYPE-C-31-M-12 (C165948). KiCad's footprint for it has the GCT part's
  pegs and shell slots with the pad row 0.38 mm further out; the footprint is swapped on the board
  with the pads kept on the old row and the body moved toward the edge, as a project copy with its
  silkscreen stopped inside the edge, like the sockets'. GCT's own USB4215 is not a drop-in.
- USB-A: TE 292303-6 (C591765), through-hole right angle on the Molex pattern.
- buttons: C&K KSC221JLFS (C221726), the same 6.2 mm J-lead family as the KSC6 drawn.
- buck inductor: Sunlord SWPA4030S4R7MT (C57269) for the prototype; the Coilcraft stays the
  production part.

Parity holds. Four clearances of 0.01 to 0.14 mm remain in the receptacle's hand-routed breakout,
where the longer pads now reach it; they are the next edit, and the export waits on them.

Co-Authored-By: Claude Fable 5.1 <noreply@anthropic.com>
Parts:
- J3: LCSC (none) -> C591765; MPN Molex 0676430910 -> TE 292303-6; Sourcing JLCPCB global sourcing -> (none)
Changed lines of the file:
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@@
 			)
 		)
-		(property "Sourcing" "JLCPCB global sourcing"
+		(property "LCSC" "C591765"
 			(at 190.5 116.84 0)
 			(show_name no)
@@
 			)
 		)
-		(property "MPN" "Molex 0676430910"
+		(property "Sourcing" ""
 			(at 190.5 116.84 0)
 			(show_name no)
+			(do_not_autoplace no)
+			(hide yes)
+			(effects
+				(font
+					(size 1.27 1.27)
+				)
+			)
+		)
+		(property "MPN" "TE 292303-6"
+			(at 190.5 116.84 0)
+			(show_name no)
