File: pcb/crossfire.kicad_sch (KiCad schematic)
At the start: 4 parts

Commit message: manual pcb finishing work
Changed lines of the file:
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@@
 		(in_pos_files yes)
 		(dnp no)
-		(property "Reference" "#PWR117"
+		(property "Reference" "#PWR03"
 			(at 76.2 173.99 0)
 			(show_name no)
@@
 			(project "crossfire"
 				(path "/4c5cdd13-4f54-43b0-affb-0ae4b9a4d279"
-					(reference "#PWR117")
+					(reference "#PWR03")
 					(unit 1)
 				)
@@
 		(in_pos_files yes)
 		(dnp no)
-		(property "Reference" "#PWR115"
+		(property "Reference" "#PWR01"
 			(at 38.1 173.99 0)
 			(show_name no)
@@
 			(project "crossfire"
 				(path "/4c5cdd13-4f54-43b0-affb-0ae4b9a4d279"
-					(reference "#PWR115")
+					(reference "#PWR01")
 					(unit 1)
 				)
@@
 		(in_pos_files yes)
 		(dnp no)
-		(property "Reference" "#PWR116"
+		(property "Reference" "#PWR02"
 			(at 57.15 173.99 0)
 			(show_name no)
@@
 			(project "crossfire"
 				(path "/4c5cdd13-4f54-43b0-affb-0ae4b9a4d279"
-					(reference "#PWR116")
+					(reference "#PWR02")
 					(unit 1)
 				)
@@
 		(in_pos_files yes)
 		(dnp no)
-		(property "Reference" "#PWR118"
+		(property "Reference" "#PWR04"
 			(at 95.25 173.99 0)
 			(show_name no)
@@
 			(project "crossfire"
 				(path "/4c5cdd13-4f54-43b0-affb-0ae4b9a4d279"
-					(reference "#PWR118")
-					(unit 1)
-				)
+					(reference "#PWR04")
+					(unit 1)
+				)
