File: pcb/crossfire.kicad_sch (KiCad schematic)
At the start: 4 parts

Commit message: every bill-of-materials line answers the assembler
The first upload to the fabricator matched the passives by value and package and failed nine
lines. Each line now carries a definite answer in the schematic, written out as columns: a
catalogue number where the part is in the catalogue -- the flash, the protection arrays, the
indicators, the ferrite, and both crystals as 10 pF parts, since the catalogue's basic crystals
are 20 pF and the processor vendor's circuit was copied with its 15 pF capacitors; a named part
and a global-sourcing note where it is not -- the buck inductor, the buttons, the USB-C receptacle
and the USB-A sockets. The debug header is marked not fitted, and the mounting holes leave the
bill and the placement file, since neither is a part.

The same fields are on the board's footprints, as an update from the schematic would put them, so
parity holds; the export writes the sourcing column; the design document carries the table.

Co-Authored-By: Claude Fable 5.1 <noreply@anthropic.com>
Parts:
- H1, H2, H3, H4: now left out of the parts list
Changed lines of the file:
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@@
 		(body_style 1)
 		(exclude_from_sim no)
-		(in_bom yes)
+		(in_bom no)
 		(on_board yes)
 		(in_pos_files yes)
@@
 		(body_style 1)
 		(exclude_from_sim no)
-		(in_bom yes)
+		(in_bom no)
 		(on_board yes)
 		(in_pos_files yes)
@@
 		(body_style 1)
 		(exclude_from_sim no)
-		(in_bom yes)
+		(in_bom no)
 		(on_board yes)
 		(in_pos_files yes)
@@
 		(body_style 1)
 		(exclude_from_sim no)
-		(in_bom yes)
-		(on_board yes)
-		(in_pos_files yes)
+		(in_bom no)
+		(on_board yes)
+		(in_pos_files yes)

Commit message: review: an indicator that lights, test points, and the sense divider gone
The green indicator could not have lit: a 3.1 V part on 3.3 V through 1 k leaves a fifth of a
milliamp. It becomes a 2.1 V yellow-green (LITEON LTST-C194KGKT, C913102) and both indicators
run through 330 ohm (C25104), about 4 mA each.

The VBUS sense divider watched the one rail the board runs from and could only ever read high.
Its two resistors, their ground, the wires, the hierarchical label and the sheet pins on both
sides are gone, GPIO17 carries a no-connect, and on the board the parts, their tracks, the
divider's 0.2 mm feed and the one via it left dangling are removed.

Eight test points go on the mcu sheet -- the PIO host pair, the processor's own USB pair, the
three rails and ground -- as bare 1 mm pads that the library keeps out of the bill and the
placement file. On the board they are parked in two rows in the open strip along the back edge,
references hidden, for the hand to place where a probe wants them; the seven connections to draw
are what the rules check lists.

Co-Authored-By: Claude Fable 5.1 <noreply@anthropic.com>
Other:
- sheet mcu ports: added none; removed VBUS_DET
- sheet upstream_data ports: added none; removed VBUS_DET
Changed lines of the file:
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@@
-	(wire
-		(pts
-			(xy 71.12 71.12) (xy 76.2 71.12)
-		)
-		(stroke
-			(width 0)
-			(type solid)
-		)
-	)
 	(wire
 		(pts
@@
 		(pts
 			(xy 152.4 139.7) (xy 157.48 139.7)
-		)
-		(stroke
-			(width 0)
-			(type solid)
-		)
-	)
-	(wire
-		(pts
-			(xy 152.4 45.72) (xy 157.48 45.72)
 		)
 		(stroke
@@
 		)
 	)
-	(label "VBUS_DET"
-		(at 76.2 71.12 0)
-		(effects
-			(font
-				(size 1.27 1.27)
-			)
-			(justify left bottom)
-		)
-	)
 	(label "P1_PWR"
 		(at 259.08 109.22 0)
@@
 	(label "P1_PWR"
 		(at 157.48 116.84 0)
-		(effects
-			(font
-				(size 1.27 1.27)
-			)
-			(justify left bottom)
-		)
-	)
-	(label "VBUS_DET"
-		(at 157.48 45.72 0)
 		(effects
 			(font
@@
 			)
 		)
-		(pin "VBUS_DET" input
-			(at 152.4 45.72 0)
-			(effects
-				(font
-					(size 1.27 1.27)
-				)
-				(justify right)
-			)
-		)
 		(pin "HUB_VBUS_DET" output
 			(at 152.4 63.5 0)
@@
 			(effects
 				(font
-					(size 1.27 1.27)
-				)
-				(justify right)
-			)
-		)
-		(pin "VBUS_DET" output
-			(at 71.12 71.12 0)
-			(effects
-				(font
