File: pcb/mcu.kicad_sch (KiCad schematic)
At the start: 32 parts, among them J1 SWD+UART, SW1 BOOT, SW2 RESET, SW3 USER, U1 RP2350A, U2 W25Q128JVS, Y1 12MHz

Commit message: manual pcb finishing work
Parts:
- renumbered C9 to C10, C12 to C11, C10 to C12, C16 to C15, C11 to C16, C1 to C17, C2 to C18, C15 to C19, C3 to C4, C4 to C5, C5 to C6, C6 to C7, C7 to C8, C8 to C9, D2 to D1, D1 to D2, J1 to J2, R4 to R10, R3 to R11, R1 to R7, R2 to R8, R5 to R9, U1 to U3
