File: pcb/mcu.kicad_sch (KiCad schematic)
At the start: 32 parts, among them J2 SWD+UART, SW1 BOOT, SW2 RESET, SW3 USER, U2 W25Q128JVS, U3 RP2350A, Y1 12MHz

Commit message: schematic: what the reference documents asked for and the drawing lacked
A pre-fab reading of the processor vendor's hardware design guide and the hub vendor's design
checklists, against the netlist pin by pin, found four omissions no rules check reports:

- the hardware USB pair had no series termination; the guide requires 27 ohm at the chip, so R21
  and R22 go between pins 51/52 and the protection array, with the chip-side stubs labelled
  MCU_D+/MCU_D- so they route as a pair and sit in the USB net class
- the crystal circuit had no series resistor on XOUT; the guide's has 1 k to keep the crystal from
  being over-driven at 3.3 V, so R23 goes between XOUT and the crystal node
- the hub's two non-removable straps were left floating; its checklist says they have no internal
  terminations and must be terminated, so R24 and R25 pull them to ground (four removable ports)
- the hub wanted a capacitor at each analogue supply pin and had one short; C45 joins its 3.3 V
  row, and C43/C44 give the processor's third DVDD pin and sixth IOVDD pin capacitors of their own

The project's net-class patterns still named the converter's old designator and the old number of
one port's VBUS net, so those nets had been in the default class; corrected. The design document
records the findings and what the same reading confirmed.

The board does not yet carry the eight parts, and its USB and XOUT tracks keep their old nets until
they are placed.

Co-Authored-By: Claude Fable 5.1 <noreply@anthropic.com>
Parts:
- added C43, C44: 100n, Capacitor_SMD:C_0402_1005Metric, symbol Device:C_Small
- added R21, R22: 27R, Resistor_SMD:R_0402_1005Metric, symbol Device:R_Small
- added R23: 1k, Resistor_SMD:R_0402_1005Metric, symbol Device:R_Small
Connections:
- net +1V1: now also C43.1
- net +3V3: now also C44.1
- net GND: now also C43.2, C44.2
- net USB_D+: now also R22.1; no longer U3.52 (USB_DP)
- net USB_D-: now also R21.1; no longer U3.51 (USB_DM)
- net at C13.1, Y1.3: now also R23.1; no longer U3.22 (XOUT)
- new net: R23.2, U3.22 (XOUT)
- new net MCU_D+: R22.2, U3.52 (USB_DP)
- new net MCU_D-: R21.2, U3.51 (USB_DM)
