File: pcb/mcu.kicad_sch (KiCad schematic)
At the start: 37 parts, among them J2 SWD+UART, SW1 BOOT, SW2 RESET, SW3 USER, U2 W25Q128JVS, U3 RP2350A, Y1 12MHz

Commit message: settle the open items by reading, pick the fabricator, and script the export
The flash is rated 133 MHz for everything but the plain read, so the QSPI divider's 120 MHz
stands. The buck's values are checked against its datasheet's table and text: the 4.7 uH stays
inside the recommended band with 0.22 A of ripple; the input capacitor becomes the same 10 uF 0805
16 V X7R part as the hub's bulk capacitor, so it still reads 10 uF with 5 V across it; the inductor
is named, a Coilcraft XEL4030-472MEC on the land already placed, chosen over the XFL part in the
same size because that one saturates below the buck's current limit. VBUS carries 10.6 uF nominal
and about 8 uF real at attach, under the 10 uF allowed. The three items that only a prototype can
answer move to their own list, with the crystals' drive level added to it.

The board goes to JLCPCB assembled: four layers with 0.2 mm vias is its standard process, it fills
and caps vias in pads, it assembles both faces and through-hole, and the four chips that matter
are in its catalogue -- their numbers are now LCSC fields on the symbols and a column in the bill
of materials. The two connectors are not, and go in as sourced or consigned parts.

scripts/export-fab.ps1 writes the Gerber and drill zip, the bill of materials and the placement
file to pcb/fab/ (untracked), after a rules check with schematic parity that refills the pours and
saves the board first, since the Gerbers are plotted from the stored fill. The first run found the
fill a step behind the last edit, which the saved board now carries.

The board still has the old C20 footprint and lacks the new fields until the schematic is pushed
to it, which is the next step before the export passes.

Co-Authored-By: Claude Fable 5.1 <noreply@anthropic.com>
Parts:
- L1: LCSC (none) -> C42411119
- U3: LCSC (none) -> C42411118; MPN (none) -> RP2350A
Changed lines of the file:
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@@
+			)
+		)
+		(property "MPN" "RP2350A"
+			(at 205.3433 186.69 0)
+			(show_name no)
+			(do_not_autoplace no)
+			(hide yes)
+			(effects
+				(font
+					(size 1.27 1.27)
+				)
+				(justify left)
+			)
+		)
+		(property "LCSC" "C42411118"
+			(at 205.3433 186.69 0)
+			(show_name no)
+			(do_not_autoplace no)
+			(hide yes)
+			(effects
+				(font
+					(size 1.27 1.27)
+				)
+				(justify left)
 			)
 		)
@@
 			(effects
 				(font
+					(size 1.27 1.27)
+				)
+				(justify right)
+			)
+		)
+		(property "LCSC" "C42411119"
+			(at 207.01 85.0899 0)
+			(show_name no)
+			(do_not_autoplace no)
+			(hide yes)
+			(effects
+				(font

Commit message: every bill-of-materials line answers the assembler
The first upload to the fabricator matched the passives by value and package and failed nine
lines. Each line now carries a definite answer in the schematic, written out as columns: a
catalogue number where the part is in the catalogue -- the flash, the protection arrays, the
indicators, the ferrite, and both crystals as 10 pF parts, since the catalogue's basic crystals
are 20 pF and the processor vendor's circuit was copied with its 15 pF capacitors; a named part
and a global-sourcing note where it is not -- the buck inductor, the buttons, the USB-C receptacle
and the USB-A sockets. The debug header is marked not fitted, and the mounting holes leave the
bill and the placement file, since neither is a part.

The same fields are on the board's footprints, as an update from the schematic would put them, so
parity holds; the export writes the sourcing column; the design document carries the table.

Co-Authored-By: Claude Fable 5.1 <noreply@anthropic.com>
Parts:
- D1: LCSC (none) -> C12624; MPN (none) -> KENTO KT-0603G
- D2: LCSC (none) -> C2286; MPN (none) -> KENTO KT-0603R
- FB1: LCSC (none) -> C2661913; MPN (none) -> Murata BLM18BD601SZ1D
- J2: MPN (none) -> 2.54 mm 1x5 header, not fitted; Sourcing (none) -> not placed; now not fitted
- SW1, SW2, SW3: MPN (none) -> C&K KSC621J LFS; Sourcing (none) -> JLCPCB global sourcing
- U2: LCSC (none) -> C97521; MPN (none) -> W25Q128JVSIQ
- Y1: LCSC (none) -> C390763; MPN (none) -> JGHC S3212000101080
Changed lines of the file:
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@@
 			)
 		)
+		(property "Sourcing" "JLCPCB global sourcing"
+			(at 135.89 115.57 0)
+			(show_name no)
+			(do_not_autoplace no)
+			(hide yes)
+			(effects
+				(font
+					(size 1.27 1.27)
+				)
+			)
+		)
+		(property "MPN" "C&K KSC621J LFS"
+			(at 135.89 115.57 0)
+			(show_name no)
+			(do_not_autoplace no)
+			(hide yes)
+			(effects
+				(font
+					(size 1.27 1.27)
+				)
+			)
+		)
 		(property "Footprint" "Button_Switch_SMD:SW_Push_1P1T_NO_CK_KSC6xxJ"
 			(at 135.89 120.65 0)
@@
 			)
 		)
+		(property "Sourcing" "JLCPCB global sourcing"
+			(at 147.32 93.98 0)
+			(show_name no)
+			(do_not_autoplace no)
+			(hide yes)
+			(effects
+				(font
+					(size 1.27 1.27)
+				)
+			)
+		)
+		(property "MPN" "C&K KSC621J LFS"
+			(at 147.32 93.98 0)
+			(show_name no)
+			(do_not_autoplace no)
+			(hide yes)
+			(effects
+				(font
+					(size 1.27 1.27)
+				)
+			)
+		)
 		(property "Footprint" "Button_Switch_SMD:SW_Push_1P1T_NO_CK_KSC6xxJ"
 			(at 147.32 99.06 0)
@@
 		(on_board yes)
 		(in_pos_files yes)
-		(dnp no)
+		(dnp yes)
 		(fields_autoplaced yes)
 		(property "Reference" "J2"
@@
 			)
 		)
+		(property "Sourcing" "not placed"
+			(at 147.32 186.69 0)
+			(show_name no)
+			(do_not_autoplace no)
+			(hide yes)
+			(effects
+				(font
+					(size 1.27 1.27)
+				)
+			)
+		)
+		(property "MPN" "2.54 mm 1x5 header, not fitted"
+			(at 147.32 186.69 0)
+			(show_name no)
+			(do_not_autoplace no)
+			(hide yes)
+			(effects
+				(font
+					(size 1.27 1.27)
+				)
+			)
+		)
 		(property "Footprint" "Connector_PinHeader_2.54mm:PinHeader_1x05_P2.54mm_Vertical"
 			(at 147.32 195.58 0)
@@
 			)
 		)
+		(property "LCSC" "C2661913"
+			(at 191.77 54.5718 0)
+			(show_name no)
+			(do_not_autoplace no)
+			(hide yes)
+			(effects
+				(font
+					(size 1.27 1.27)
+				)
+				(justify left)
+			)
+		)
+		(property "MPN" "Murata BLM18BD601SZ1D"
+			(at 191.77 54.5718 0)
+			(show_name no)
+			(do_not_autoplace no)
+			(hide yes)
+			(effects
+				(font
+					(size 1.27 1.27)
+				)
+				(justify left)
+			)
+		)
 		(property "Footprint" "Inductor_SMD:L_0603_1608Metric"
 			(at 189.23 53.34 0)
@@
 			)
 		)
+		(property "Sourcing" "JLCPCB global sourcing"
+			(at 261.62 184.15 0)
+			(show_name no)
+			(do_not_autoplace no)
+			(hide yes)
+			(effects
+				(font
+					(size 1.27 1.27)
+				)
+			)
+		)
+		(property "MPN" "C&K KSC621J LFS"
+			(at 261.62 184.15 0)
+			(show_name no)
+			(do_not_autoplace no)
+			(hide yes)
+			(effects
+				(font
+					(size 1.27 1.27)
+				)
+			)
+		)
 		(property "Footprint" "Button_Switch_SMD:SW_Push_1P1T_NO_CK_KSC6xxJ"
 			(at 261.62 189.23 0)
@@
 			)
 		)
+		(property "LCSC" "C97521"
+			(at 96.52 144.1449 0)
+			(show_name no)
+			(do_not_autoplace no)
+			(hide yes)
+			(effects
+				(font
+					(size 1.27 1.27)
+				)
+				(justify left)
+			)
+		)
+		(property "MPN" "W25Q128JVSIQ"
+			(at 96.52 144.1449 0)
+			(show_name no)
+			(do_not_autoplace no)
+			(hide yes)
+			(effects
+				(font
+					(size 1.27 1.27)
+				)
+				(justify left)
+			)
+		)
 		(property "Footprint" "Package_SO:SOIC-8_5.3x5.3mm_P1.27mm"
 			(at 110.49 142.24 0)
@@
 			)
 		)
+		(property "LCSC" "C390763"
+			(at 147.32 161.29 0)
+			(show_name no)
+			(do_not_autoplace no)
+			(hide yes)
+			(effects
+				(font
+					(size 1.27 1.27)
+				)
+			)
+		)
+		(property "MPN" "JGHC S3212000101080"
+			(at 147.32 161.29 0)
+			(show_name no)
+			(do_not_autoplace no)
+			(hide yes)
+			(effects
+				(font
+					(size 1.27 1.27)
+				)
+			)
+		)
 		(property "Footprint" "Crystal:Crystal_SMD_3225-4Pin_3.2x2.5mm"
 			(at 147.32 165.1 0)
@@
 			)
 		)
+		(property "LCSC" "C2286"
+			(at 272.9865 156.21 0)
+			(show_name no)
+			(do_not_autoplace no)
+			(hide yes)
+			(effects
+				(font
+					(size 1.27 1.27)
+				)
+			)
+		)
+		(property "MPN" "KENTO KT-0603R"
+			(at 272.9865 156.21 0)
+			(show_name no)
+			(do_not_autoplace no)
+			(hide yes)
+			(effects
+				(font
+					(size 1.27 1.27)
+				)
+			)
+		)
 		(property "Footprint" "LED_SMD:LED_0603_1608Metric"
 			(at 273.05 160.02 0)
@@
 			(effects
 				(font
+					(size 1.27 1.27)
+				)
+			)
+		)
+		(property "LCSC" "C12624"
+			(at 261.5565 168.91 0)
+			(show_name no)
+			(do_not_autoplace no)
+			(hide yes)
+			(effects
+				(font
+					(size 1.27 1.27)
+				)
+			)
+		)
+		(property "MPN" "KENTO KT-0603G"
+			(at 261.5565 168.91 0)
+			(show_name no)
+			(do_not_autoplace no)
+			(hide yes)
+			(effects
+				(font

Commit message: the four sourced lines become catalogue parts
Global sourcing turned out to be a pre-purchase into one's own library, three to four weeks and an
inspection fee per kind of connector or switch, so the connectors, the buttons and the prototype's
inductor come from the catalogue instead, each checked against a drawing rather than a part page:

- USB-C: Korean Hroparts TYPE-C-31-M-12 (C165948). KiCad's footprint for it has the GCT part's
  pegs and shell slots with the pad row 0.38 mm further out; the footprint is swapped on the board
  with the pads kept on the old row and the body moved toward the edge, as a project copy with its
  silkscreen stopped inside the edge, like the sockets'. GCT's own USB4215 is not a drop-in.
- USB-A: TE 292303-6 (C591765), through-hole right angle on the Molex pattern.
- buttons: C&K KSC221JLFS (C221726), the same 6.2 mm J-lead family as the KSC6 drawn.
- buck inductor: Sunlord SWPA4030S4R7MT (C57269) for the prototype; the Coilcraft stays the
  production part.

Parity holds. Four clearances of 0.01 to 0.14 mm remain in the receptacle's hand-routed breakout,
where the longer pads now reach it; they are the next edit, and the export waits on them.

Co-Authored-By: Claude Fable 5.1 <noreply@anthropic.com>
Parts:
- SW1, SW2, SW3: LCSC (none) -> C221726; MPN C&K KSC621J LFS -> C&K KSC221JLFS; Sourcing JLCPCB global sourcing -> (none)
Changed lines of the file:
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@@
 			)
 		)
-		(property "Sourcing" "JLCPCB global sourcing"
+		(property "LCSC" "C221726"
 			(at 135.89 115.57 0)
 			(show_name no)
@@
 			)
 		)
-		(property "MPN" "C&K KSC621J LFS"
+		(property "Sourcing" ""
+			(at 135.89 115.57 0)
+			(show_name no)
+			(do_not_autoplace no)
+			(hide yes)
+			(effects
+				(font
+					(size 1.27 1.27)
+				)
+			)
+		)
+		(property "MPN" "C&K KSC221JLFS"
 			(at 135.89 115.57 0)
 			(show_name no)
@@
 			)
 		)
-		(property "Sourcing" "JLCPCB global sourcing"
+		(property "LCSC" "C221726"
+			(at 147.32 93.98 0)
+			(show_name no)
+			(do_not_autoplace no)
+			(hide yes)
+			(effects
+				(font
+					(size 1.27 1.27)
+				)
+			)
+		)
+		(property "Sourcing" ""
 			(at 147.32 93.98 0)
 			(show_name no)
@@
 			)
 		)
-		(property "MPN" "C&K KSC621J LFS"
+		(property "MPN" "C&K KSC221JLFS"
 			(at 147.32 93.98 0)
 			(show_name no)
@@
 			)
 		)
-		(property "Sourcing" "JLCPCB global sourcing"
+		(property "LCSC" "C221726"
+			(at 261.62 184.15 0)
+			(show_name no)
+			(do_not_autoplace no)
+			(hide yes)
+			(effects
+				(font
+					(size 1.27 1.27)
+				)
+			)
+		)
+		(property "Sourcing" ""
 			(at 261.62 184.15 0)
 			(show_name no)
@@
 			)
 		)
-		(property "MPN" "C&K KSC621J LFS"
+		(property "MPN" "C&K KSC221JLFS"
 			(at 261.62 184.15 0)
 			(show_name no)

Commit message: pin the passives the matcher got wrong, and close the receptacle's clearances
The fabricator's matcher put the 1 uF on a 01005 part, found nothing for the 4.7 uF or the 27 ohm,
and the ferrite's first choice ran out, so those lines carry catalogue numbers now: Samsung
CL05A105KO5NNNC and CL05A475MP5NRNC (10 V, the basic part), UNI-ROYAL 0402WGF270JTCE, Murata
BLM18KG601SN1D. The 5.1 k CC pull-downs are left to any 1 % part with stock, the specification
allowing ten percent there. The four clearances the receptacle swap left in its breakout are
closed by hand. The rules check is clean with parity and the fab files are regenerated.

Co-Authored-By: Claude Fable 5.1 <noreply@anthropic.com>
Parts:
- C15: LCSC (none) -> C29266; MPN (none) -> Samsung CL05A105KO5NNNC; Voltage 6.3V -> 16V
- C17, C4: LCSC (none) -> C23733; MPN (none) -> Samsung CL05A475MP5NRNC; Voltage 6.3V -> 10V
- FB1: LCSC C2661913 -> C85833; MPN Murata BLM18BD601SZ1D -> Murata BLM18KG601SN1D
- R21, R22: LCSC (none) -> C25100; MPN (none) -> UNI-ROYAL 0402WGF270JTCE
Changed lines of the file:
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@@
 			)
 		)
+		(property "LCSC" "C25100"
+			(at 167.64 132.08 90)
+			(show_name no)
+			(do_not_autoplace no)
+			(hide yes)
+			(effects
+				(font
+					(size 1.27 1.27)
+				)
+			)
+		)
+		(property "MPN" "UNI-ROYAL 0402WGF270JTCE"
+			(at 167.64 132.08 90)
+			(show_name no)
+			(do_not_autoplace no)
+			(hide yes)
+			(effects
+				(font
+					(size 1.27 1.27)
+				)
+			)
+		)
 		(property "Footprint" "Resistor_SMD:R_0402_1005Metric"
 			(at 167.64 127 0)
@@
 			)
 		)
+		(property "LCSC" "C23733"
+			(at 226.06 87.6362 0)
+			(show_name no)
+			(do_not_autoplace no)
+			(hide yes)
+			(effects
+				(font
+					(size 1.27 1.27)
+				)
+				(justify left)
+			)
+		)
+		(property "MPN" "Samsung CL05A475MP5NRNC"
+			(at 226.06 87.6362 0)
+			(show_name no)
+			(do_not_autoplace no)
+			(hide yes)
+			(effects
+				(font
+					(size 1.27 1.27)
+				)
+				(justify left)
+			)
+		)
 		(property "Footprint" "Capacitor_SMD:C_0402_1005Metric"
 			(at 223.52 86.36 0)
@@
 			)
 		)
-		(property "Voltage" "6.3V"
+		(property "Voltage" "10V"
 			(at 226.822 89.408 0)
 			(hide yes)
@@
 			)
 		)
-		(property "LCSC" "C2661913"
+		(property "LCSC" "C85833"
 			(at 191.77 54.5718 0)
 			(show_name no)
@@
 			)
 		)
-		(property "MPN" "Murata BLM18BD601SZ1D"
+		(property "MPN" "Murata BLM18KG601SN1D"
 			(at 191.77 54.5718 0)
 			(show_name no)
@@
 			)
 		)
+		(property "LCSC" "C29266"
+			(at 182.88 95.2562 0)
+			(show_name no)
+			(do_not_autoplace no)
+			(hide yes)
+			(effects
+				(font
+					(size 1.27 1.27)
+				)
+				(justify left)
+			)
+		)
+		(property "MPN" "Samsung CL05A105KO5NNNC"
+			(at 182.88 95.2562 0)
+			(show_name no)
+			(do_not_autoplace no)
+			(hide yes)
+			(effects
+				(font
+					(size 1.27 1.27)
+				)
+				(justify left)
+			)
+		)
 		(property "Footprint" "Capacitor_SMD:C_0402_1005Metric"
 			(at 180.34 93.98 0)
@@
 			)
 		)
-		(property "Voltage" "6.3V"
+		(property "Voltage" "16V"
 			(at 183.642 97.028 0)
 			(hide yes)
@@
 			)
 		)
+		(property "LCSC" "C23733"
+			(at 73.66 72.3962 0)
+			(show_name no)
+			(do_not_autoplace no)
+			(hide yes)
+			(effects
+				(font
+					(size 1.27 1.27)
+				)
+				(justify left)
+			)
+		)
+		(property "MPN" "Samsung CL05A475MP5NRNC"
+			(at 73.66 72.3962 0)
+			(show_name no)
+			(do_not_autoplace no)
+			(hide yes)
+			(effects
+				(font
+					(size 1.27 1.27)
+				)
+				(justify left)
+			)
+		)
 		(property "Footprint" "Capacitor_SMD:C_0402_1005Metric"
 			(at 71.12 71.12 0)
@@
 			)
 		)
-		(property "Voltage" "6.3V"
+		(property "Voltage" "10V"
 			(at 73.914 73.66 0)
 			(hide yes)
@@
 			(effects
 				(font
+					(size 1.27 1.27)
+				)
+			)
+		)
+		(property "LCSC" "C25100"
+			(at 167.64 121.92 90)
+			(show_name no)
+			(do_not_autoplace no)
+			(hide yes)
+			(effects
+				(font
+					(size 1.27 1.27)
+				)
+			)
+		)
+		(property "MPN" "UNI-ROYAL 0402WGF270JTCE"
+			(at 167.64 121.92 90)
+			(show_name no)
+			(do_not_autoplace no)
+			(hide yes)
+			(effects
+				(font

Commit message: review: an indicator that lights, test points, and the sense divider gone
The green indicator could not have lit: a 3.1 V part on 3.3 V through 1 k leaves a fifth of a
milliamp. It becomes a 2.1 V yellow-green (LITEON LTST-C194KGKT, C913102) and both indicators
run through 330 ohm (C25104), about 4 mA each.

The VBUS sense divider watched the one rail the board runs from and could only ever read high.
Its two resistors, their ground, the wires, the hierarchical label and the sheet pins on both
sides are gone, GPIO17 carries a no-connect, and on the board the parts, their tracks, the
divider's 0.2 mm feed and the one via it left dangling are removed.

Eight test points go on the mcu sheet -- the PIO host pair, the processor's own USB pair, the
three rails and ground -- as bare 1 mm pads that the library keeps out of the bill and the
placement file. On the board they are parked in two rows in the open strip along the back edge,
references hidden, for the hand to place where a probe wants them; the seven connections to draw
are what the rules check lists.

Co-Authored-By: Claude Fable 5.1 <noreply@anthropic.com>
Parts:
- added TP1, TP2, TP3, TP4, TP5, TP6, TP7, TP8: TestPoint, TestPoint:TestPoint_Pad_1.0x1.0mm, symbol Connector:TestPoint
- D1: value green -> yellow-green; LCSC C12624 -> C913102; MPN KENTO KT-0603G -> LITEON LTST-C194KGKT; Vf (none) -> 2.1V
- R10, R11: value 1k -> 330R; LCSC (none) -> C25104; MPN (none) -> UNI-ROYAL 0402WGF3300TCE
Connections:
- net +1V1: now also TP7.1
- net +3V3: now also TP6.1
- net GND: now also TP8.1
- net PIO_D+: now also TP1.1
- net PIO_D-: now also TP2.1
- net USB_D+: now also TP3.1
- net USB_D-: now also TP4.1
- net VBUS_DET: no longer names the net of U3.28 (GPIO17)
- new net +5V: TP5.1
- no-connect marks 18 -> 19

Commit message: C44 comes out: the sixth IOVDD pin shares the regulator's input capacitor
There is no room at that pin for a capacitor of its own, the 4.7 uF on VREG_VIN sits 2.5 mm from
it on the same net, and the vendor's own board shares a capacitor between two pins in exactly
that situation. The capacitor, its wires and junction leave the sheet; the footprint, its stub,
its via and the segment the stub left behind leave the board. The design document records the
reversal next to the addition.

Co-Authored-By: Claude Fable 5.1 <noreply@anthropic.com>
Parts:
- removed C44: 100n, Capacitor_SMD:C_0402_1005Metric, symbol Device:C_Small
Changed lines of the file:
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@@
 	)
 	(junction
-		(at 142.24 67.31)
-		(diameter 0)
-		(color 0 0 0 0)
-	)
-	(junction
 		(at 101.6 76.2)
 		(diameter 0)
@@
 	(wire
 		(pts
-			(xy 152.4 67.31) (xy 152.4 68.58)
-		)
-		(stroke
-			(width 0)
-			(type default)
-		)
-	)
-	(wire
-		(pts
 			(xy 228.6 101.6) (xy 233.68 101.6)
 		)
@@
 	(wire
 		(pts
-			(xy 142.24 76.2) (xy 152.4 76.2)
-		)
-		(stroke
-			(width 0)
-			(type default)
-		)
-	)
-	(wire
-		(pts
 			(xy 91.44 67.31) (xy 101.6 67.31)
 		)
@@
 	(wire
 		(pts
-			(xy 152.4 73.66) (xy 152.4 76.2)
-		)
-		(stroke
-			(width 0)
-			(type default)
-		)
-	)
-	(wire
-		(pts
 			(xy 265.43 137.16) (xy 265.43 147.32)
 		)
@@
 	(wire
 		(pts
-			(xy 142.24 67.31) (xy 152.4 67.31)
-		)
-		(stroke
-			(width 0)
-			(type default)
-		)
-	)
-	(wire
-		(pts
 			(xy 167.64 165.1) (xy 149.86 165.1)
 		)
@@
 					(unit 1)
 				)
-			)
-		)
-	)
-	(symbol
-		(lib_id "Device:C_Small")
-		(at 152.4 71.12 0)
-		(unit 1)
-		(body_style 1)
-		(exclude_from_sim no)
-		(in_bom yes)
-		(on_board yes)
-		(in_pos_files yes)
-		(dnp no)
-		(fields_autoplaced yes)
-		(property "Reference" "C44"
-			(at 154.94 69.8562 0)
-			(show_name no)
-			(do_not_autoplace no)
-			(effects
-				(font
-					(size 1.27 1.27)
-				)
-				(justify left)
-			)
-		)
-		(property "Value" "100n"
-			(at 154.94 72.3962 0)
-			(show_name no)
-			(do_not_autoplace no)
-			(effects
-				(font
-					(size 1.27 1.27)
-				)
-				(justify left)
-			)
-		)
-		(property "Footprint" "Capacitor_SMD:C_0402_1005Metric"
-			(at 152.4 71.12 0)
-			(hide yes)
-			(show_name no)
-			(do_not_autoplace no)
-			(effects
-				(font
-					(size 1.27 1.27)
-				)
-			)
-		)
-		(property "Datasheet" ""
-			(at 152.4 71.12 0)
-			(hide yes)
-			(show_name no)
-			(do_not_autoplace no)
-			(effects
-				(font
-					(size 1.27 1.27)
-				)
-			)
-		)
-		(property "Description" ""
-			(at 152.4 71.12 0)
-			(hide yes)
-			(show_name no)
-			(do_not_autoplace no)
-			(effects
-				(font
-					(size 1.27 1.27)
-				)
-			)
-		)
-		(property "Voltage" "16V"
-			(at 155.194 73.66 0)
-			(hide yes)
-			(show_name no)
-			(do_not_autoplace no)
-			(effects
-				(font
-					(size 1.27 1.27)
-				)
-			)
-		)
-		(property "Dielectric" "X7R"
-			(at 155.194 73.66 0)
-			(hide yes)
-			(show_name no)
-			(do_not_autoplace no)
-			(effects
-				(font
-					(size 1.27 1.27)
-				)
-			)
-		)
-		(pin "1"
-		)
-		(pin "2"
-		)
-		(instances
-			(project "crossfire"
-				(path "/4c5cdd13-4f54-43b0-affb-0ae4b9a4d279/4cdbbf45-e559-4c12-a33c-465c1e579944"
-					(reference "C44")
-					(unit 1)
-				)
