File: pcb/crossfire.kicad_pcb (KiCad board)
At the start: 4 copper layers, 100 x 54 mm, 95 parts, among them J1 SWD+UART, J2 USB_A, J3 USB_A, J4 USB_A, J5 USB_A, J6 USB-C, SW1 BOOT, SW2 RESET, SW3 USER, U1 RP2350A, U10 TPS2065C, U11 USBLC6-2SC6, U12 USBLC6-2SC6, U14 AP63203WU, U2 W25Q128JVS, U3 USB2514B, U4 TPS2065C, U5 USBLC6-2SC6, U6 TPS2065C, U7 USBLC6-2SC6, U8 TPS2065C, U9 USBLC6-2SC6, Y1 12MHz, Y2 24MHz

Commit message: manual routing and finishing work on the pcb
Parts:
- moved C62 54.8 mm to (164.8, 77.5), turned to 0 degrees
- moved H3 3.45 mm to (123.0, 91.0)
- moved H4 3.15 mm to (173.9, 91.3)
- moved C6 1.56 mm to (138.7, 69.0)
- moved C4 0.45 mm to (143.6, 67.0)
- moved C3 0.12 mm to (135.3, 69.8)
Routing:
- net +1V1: track 40.2 -> 32.5 mm
- net +5V: track 30.3 -> 25.7 mm, vias 14 -> 13
- net +3V3: track 50.8 -> 48.8 mm
- net Net-(R1-Pad1): track 38.2 -> 39.2 mm
- net GND: track 14.0 -> 13.3 mm, vias 64 -> 66
- net /USB_D+: track 30.5 -> 30.0 mm

Commit message: more manual PCB cleanup work
Parts:
- moved C38 1.86 mm to (165.1, 62.2), turned to 0 degrees
- moved C51 1.53 mm to (128.1, 67.2), turned to -90 degrees
- moved C2 0.73 mm to (143.4, 65.0)
- moved C37 0.72 mm to (165.1, 65.2), turned to 0 degrees
- moved C5 0.54 mm to (143.4, 63.1)
- moved C31 0.32 mm to (165.1, 63.2)
- moved C4 0.11 mm to (143.4, 67.0)
Routing:
- net +3V3: track 48.8 -> 42.9 mm
- net Net-(J2-VBUS): track 19.9 -> 14.3 mm
- net /P3_OC: track 26.6 -> 24.3 mm
- net +1V1: track 32.5 -> 30.5 mm
- net Net-(U14-SW): track 8.69 -> 7.49 mm
- net GND: track 13.3 -> 12.4 mm, vias 66 -> 64
- net /CC2_SENSE: track 31.1 -> 31.7 mm

Commit message: manual pcb finishing work
Parts:
- C60, C61, C62, C63, R30, R34, U10, U4, U6, U8: moved to B.Cu
- U11, U5, U7, U9: moved to F.Cu
- moved C34 33.7 mm to (124.8, 52.6), turned to -90 degrees
- moved C9 14.6 mm to (139.9, 59.2), turned to 90 degrees
- moved U11 8.16 mm to (186.4, 80.5), turned to -90 degrees
- moved U9 8.06 mm to (161.1, 80.7), turned to -90 degrees
- moved C51 6.36 mm to (133.2, 63.5), turned to 90 degrees
- moved C63 5.23 mm to (193.1, 81.8), turned to 90 degrees
- moved C61 5.10 mm to (142.1, 81.5), turned to 90 degrees
- moved U6 4.30 mm to (139.4, 81.0), turned to 0 degrees
- moved C62 4.26 mm to (167.5, 80.8), turned to 90 degrees
- moved C52 3.87 mm to (133.2, 65.8), turned to 180 degrees
- moved C13 2.84 mm to (137.8, 54.9)
- moved Y1 2.84 mm to (140.4, 55.0)
- moved R21 2.57 mm to (159.8, 58.2), turned to -90 degrees
- moved C10 2.11 mm to (138.9, 74.8)
- moved R30 1.93 mm to (108.2, 68.7), turned to 90 degrees
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Routing:
- net /P3_D+: track 30.1 -> 13.8 mm, vias 1 -> 0
- net /P3_D-: track 28.5 -> 13.9 mm, vias 1 -> 0
- net /P2_D+: track 41.0 -> 32.0 mm, vias 1 -> 0
- net /P2_PWR: track 39.9 -> 31.2 mm, vias 2 -> 1
- net /P4_OC: track 43.1 -> 36.0 mm, vias 0 -> 1
- net /P2_D-: track 39.2 -> 32.8 mm, vias 1 -> 0
- net Net-(J4-VBUS): track 17.2 -> 11.0 mm, vias 1 -> 3
- net Net-(J5-VBUS): track 17.1 -> 11.3 mm, vias 1 -> 3
- net /P1_D+: track 61.8 -> 56.8 mm, vias 1 -> 0
- net /P4_D-: track 34.8 -> 30.1 mm, vias 1 -> 0
- net /P4_D+: track 36.4 -> 32.0 mm, vias 1 -> 0
- net Net-(U1-GPIO15): track 64.9 -> 60.6 mm
- net /P3_OC: track 24.3 -> 20.2 mm, vias 2 -> 1
- net /USB_D-: track 32.2 -> 28.3 mm
- net Net-(U1-XIN): track 6.51 -> 9.77 mm
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
Commit message: more pcb changes
Parts:
- moved C36 1.00 mm to (160.6, 67.8)
Routing:
- net +3V3: track 46.0 -> 45.2 mm
